File: v1/v1.kicad_sch (KiCad schematic)
At the start: 11 parts, among them J1 DE9_Socket, J2 Screw_Terminal_01x02, J7 Conn_02x20_Odd_Even, U1 MAX3232

Commit message: fixed footprints on v1
Parts:
- C1, C2: footprint Capacitor_SMD:C_0201_0603Metric -> Capacitor_SMD:C_0402_1005Metric
- D1: footprint Diode_SMD:D_0201_0603Metric -> Diode_SMD:D_SMB
Changed lines of the file:
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@@
 			)
 		)
-		(property "Footprint" "Capacitor_SMD:C_0201_0603Metric"
+		(property "Footprint" "Capacitor_SMD:C_0402_1005Metric"
 			(at 92.71 153.67 0)
 			(hide yes)
@@
 			)
 		)
-		(property "Footprint" "Capacitor_SMD:C_0201_0603Metric"
+		(property "Footprint" "Capacitor_SMD:C_0402_1005Metric"
 			(at 44.45 153.67 0)
 			(hide yes)
@@
 			)
 		)
-		(property "Footprint" "Diode_SMD:D_0201_0603Metric"
+		(property "Footprint" "Diode_SMD:D_SMB"
 			(at 58.42 151.13 0)
 			(hide yes)
