File: v1/v1.kicad_pcb (KiCad board)
At the start: 2 copper layers, 65.5 x 30 mm, 15 parts, among them J1 DE9_Socket, J2 Screw_Terminal_01x02, J3 Conn_01x02_Pin, J4 Conn_01x02_Pin, J5 Conn_01x02_Pin, J6 Conn_01x02_Pin, J7 Conn_02x20_Odd_Even, U1 MAX3232

Commit message: fixed footprints on v1
Parts:
- C1, C2: footprint Capacitor_SMD:C_0201_0603Metric -> Capacitor_SMD:C_0402_1005Metric
- D1: footprint Diode_SMD:D_0201_0603Metric -> Diode_SMD:D_SMB
- moved C1 3.47 mm to (132.5, 91.1), turned to 0 degrees
- moved J2 2.51 mm to (130.5, 82.5)
- moved D1 1.54 mm to (127.8, 93.0)
Routing:
- net /TPS54560/VIN: track 15.1 -> 12.2 mm
- net Net-(D1-A): track 9.43 -> 7.96 mm

Commit message: adding more electrical isolation
Parts:
- C1, C2: moved to B.Cu
- moved D1 10.5 mm to (128.0, 82.5)
- moved J2 9.35 mm to (127.0, 91.2), turned to 0 degrees
- moved U1 6.14 mm to (79.5, 92.5)
- moved C2 1.66 mm to (84.0, 83.5)
- moved C1 1.54 mm to (134.0, 91.5), turned to -90 degrees
Routing:
- net Net-(U1-R1IN): track 17.7 -> 10.6 mm
- net Net-(U1-T1OUT): track 19.0 -> 12.2 mm
- net Net-(J7-Pin_1): track 6.96 -> 13.1 mm
- net /lvlTx: track 13.0 -> 19.1 mm
- net /lvlRx: track 17.1 -> 23.2 mm
- net /TPS54560/VIN: track 12.2 -> 6.63 mm
- net Net-(D1-A): track 7.96 -> 13.2 mm
- net GND: vias 3 -> 2
