File: Hack Week/v3/v3.kicad_sch (KiCad schematic)
At the start: 10 parts, among them J2 Screw_Terminal_01x02, J3 Conn_01x04_Socket, J7 Conn_02x20_Odd_Even

Commit message: added new v3 board
Parts:
- J3: footprint (none) -> Connector_PinSocket_2.54mm:PinSocket_1x04_P2.54mm_Vertical
Changed lines of the file:
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@@
 			)
 		)
-		(property "Footprint" ""
+		(property "Footprint" "Connector_PinSocket_2.54mm:PinSocket_1x04_P2.54mm_Vertical"
 			(at 120.65 111.76 0)
 			(hide yes)
