File: Hack Week/v3_rs485/v3_rs485.kicad_sch (KiCad schematic)
At the start: 3 parts, among them J1 DE9_Socket, J2 Conn_01x04_Socket, U1 MAX3485

Commit message: changed DB9 connectors + added RS485
Parts:
- removed J1: DE9_Socket, Connector_Dsub:DSUB-9_Socket_EdgeMount_P2.77mm, symbol Connector:DE9_Socket
- added J3: LD09S33E4GV00LF, Connector_Pin:AMPHENOL_LD09S33E4GV00LF, symbol LD09S33E4GV00LF:LD09S33E4GV00LF
- J2: footprint (none) -> Connector_PinSocket_2.54mm:PinSocket_1x04_P2.54mm_Vertical
Connections:
- net GND: now also J3.5, J3.SH1 (SHIELD), J3.SH2 (SHIELD)
- net at U1.6 (A): now also J3.3
- net at U1.7 (B): now also J3.8
- no-connect marks 3 -> 6
