File: Hack Week/v3_usb/v3_usb.kicad_pcb (KiCad board)
At the start: 2 copper layers, 13.4 x 4.5 mm, 7 parts, among them J1 USB_C_Receptacle, J2 Conn_01x04_Socket, U1 FT230XQ

Commit message: changes made
Parts:
- removed J1: USB_C_Receptacle, Connector_USB:USB_C_Receptacle_Amphenol_12401948E412A
- removed R1, R2: 5.1k, Resistor_SMD:R_0603_1608Metric
- added J3: USB_A, Connector_USB:USB_A_Wuerth_614004134726_Horizontal, F.Cu at (98.5, 67.0)
- moved J2 26.9 mm to (115.5, 63.7)
- moved C2 25.2 mm to (108.2, 63.0)
- moved U1 24.8 mm to (110.0, 67.0), turned to -90 degrees
- moved C1 15.3 mm to (108.5, 70.5)
Connections:
- C1 pad 2: Net-(U1-3V3OUT) -> /Power
- U1 pad 1: Net-(U1-3V3OUT) -> /Power
- U1 pad 8: Net-(U1-3V3OUT) -> /Power
Routing:
- net /Power: track 0.00 -> 25.5 mm, vias 0 -> 1
- net /USBDM: track 0.00 -> 8.37 mm
- net /USBDP: track 0.00 -> 6.39 mm
- net /lvlRx: track 0.00 -> 5.95 mm, vias 0 -> 1
- net /lvlTx: track 0.00 -> 4.69 mm
- net GND: track 0.00 -> 4.44 mm, vias 0 -> 1
- added copper zone on B.Cu, net GND
- added copper zone on F.Cu, net GND
Other:
- board size 13.4 x 4.5 mm -> 32 x 12 mm
