File: Hack Week/v3_usb/v3_usb.kicad_sch (KiCad schematic)
At the start: 7 parts, among them J1 USB_C_Receptacle, J2 Conn_01x04_Socket, U1 FT230XQ

Commit message: changes made
Parts:
- removed J1: USB_C_Receptacle, Connector_USB:USB_C_Receptacle_Amphenol_12401948E412A, symbol Connector:USB_C_Receptacle
- removed R1, R2: 5.1k, Resistor_SMD:R_0603_1608Metric, symbol Device:R
- added J3: USB_A, Connector_USB:USB_A_Wuerth_614004134726_Horizontal, symbol Connector:USB_A
Connections:
- net GND: now also J3.4 (GND), J3.SH (Shield)
- net Power: now also C1.2, U1.1 (VCCIO), U1.8 (3V3OUT)
- net USBDM: now also J3.2 (D-)
- net USBDP: now also J3.3 (D+)
- no-connect marks 17 -> 8
